File: pcb/Garage_Door_Controller.sch (EAGLE design)
At the start: 34 parts, among them Q1 MMBT2222AL, Q2 MMBT2222AL

Commit message: Rev A schematics and board layout
Parts:
- USB: value USB_MICRO-B_10118193-0001LF -> USB_MICRO-B_47346-0001; device Connectors:USB_MICRO-B_10118193-0001LF -> Connectors:USB_MICRO-B_47346-0001
- renumbered DOWNLOAD to PROG, LED1 to LED_R, LED2 to LED_Y, LED3 to LED_G, PWR_LED to LED_PWR
Connections:
- removed net IO13: ESP32.IO13, GPIO.4
- removed net IO16_RELAY: ESP32.IO16, RELAY.3
- removed net IO21_LED_R: ESP32.IO21, R9.2
- removed net IO23_LED_G: ESP32.IO23, R11.2
- removed net IO25_TEMP: ESP32.IO25, TEMP.3
- removed net IO27: ESP32.IO27, GPIO.6
- new net IO13_RELAY: ESP32.IO13, RELAY.3
- new net IO21_LED_G: ESP32.IO21, R11.2
- new net IO23_LED_R: ESP32.IO23, R9.2
- new net IO25: ESP32.IO25, GPIO.6
- new net IO27_TEMP: ESP32.IO27, TEMP.3
- net +3V3: now also GPIO.3, GPIO.4; no longer GPIO.2
- net +5V: now also GPIO.2, USB.VBUS; no longer GPIO.3, USB.VUSB
- net CTS: now also PROG.4; no longer PROG.5
- net DSR: now also PROG.5; no longer PROG.4
- net IO32: now also GPIO.8; no longer GPIO.7
- net IO33: now also GPIO.7; no longer GPIO.8
- net RXD0: now also PROG.3; no longer PROG.2
- net TXD0: now also PROG.2; no longer PROG.3
Other:
- moved on the sheet: USB
